File: boards/circle_of_life/circle_of_life.kicad_sch (KiCad schematic)
At the start: 99 parts, among them IC1 ESP32-WROOM-32E-N8R2, IC2 TC1262-3.3VDB, IC3 TPS565242DRLR, IC4 LT3922EUFD#PBF, J1 Water Pump Connector, J10 Conn_01x12_Pin, J2 Servo Motor Connector, J3 Power Connector, J4 pH Sensor, J5 Water Flow Sensor Connector, J6 Temperature Sensor Connector, J7 UART Programmer, J8 JTAG Connector, Q1 RQ5E030AJTCL, Q2 PMOS, SW1 RESET, SW2 BOOT

Commit message: started assigning footprints
Parts:
- added D5, D6, D7: LED, symbol Device:LED
- added R26, R27, R28: 270, symbol Device:R
- C1, C10, C2, C23, C30, C35, C39, C41: footprint (none) -> SamacSys_Parts:CAPC2012X135N
- C11, C14, C16, C28, C31, C32, C34, C38, C5, C8: footprint (none) -> SamacSys_Parts:CAPAE630X800N
- C15: value 0.1u -> 0.1uF; footprint (none) -> SamacSys_Parts:CAPAE630X800N
- C18: value 1u -> 1uF; footprint (none) -> SamacSys_Parts:CAPC2012X135N
- D4: footprint Diode_SMD:D_SMA -> SamacSys_Parts:DIOM5436X247N
- F2: footprint FUSC6125X236N -> SamacSys_Parts:FUSC6125X236N
- J3: footprint 694108301002 -> SamacSys_Parts:694108301002
- L1: value L -> 4.7µH
- Q1: footprint SOT95P280X100-3N -> SamacSys_Parts:SOT95P280X100-3N
Connections:
- net GND: now also D5.1 (K), D6.1 (K), D7.1 (K)
- net IO0: no longer IC1.25 (IO0)
- net IO16: no longer IC1.27 (IO16)
- net IO4: no longer IC1.26 (IO4)
- new net: D7.2 (A), R28.1
- new net: D5.2 (A), R26.2
- new net: D6.2 (A), R27.1
- new net FLOW_FAULT: IC1.26 (IO4), R27.2
- new net PH_FAULT: IC1.25 (IO0), R26.1
- new net TEMP_FAULT: IC1.27 (IO16), R28.2
Other:
- note removed: "Missing capacitors"
- moved on the sheet: C38, C39, R24, R25, SW1

Commit message: more footprint assignments
Parts:
- D1: footprint DIOM7959X262N -> SamacSys_Parts:DIOM7959X262N
- D3: footprint SOD3716X145N -> SamacSys_Parts:SOD3716X145N
- LED1, LED10, LED3, LED5, LED9: footprint ASMWLL00NKM0E -> SamacSys_Parts:ASMWLL00NKM0E
- LED2, LED4, LED6, LED7, LED8: footprint ASMWLL00NKM0E -> SamacSys_Parts:ASMWL300AFH0E
Changed lines of the file:
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@@
 			)
 		)
-		(property "Footprint" "ASMWLL00NKM0E"
+		(property "Footprint" "SamacSys_Parts:ASMWLL00NKM0E"
 			(at 214.63 171.78 0)
 			(effects
@@
 			)
 		)
-		(property "Footprint" "ASMWLL00NKM0E"
+		(property "Footprint" "SamacSys_Parts:ASMWL300AFH0E"
 			(at 234.95 147.65 0)
 			(effects
@@
 			)
 		)
-		(property "Footprint" "ASMWLL00NKM0E"
+		(property "Footprint" "SamacSys_Parts:ASMWL300AFH0E"
 			(at 194.31 147.65 0)
 			(effects
@@
 			)
 		)
-		(property "Footprint" "ASMWLL00NKM0E"
+		(property "Footprint" "SamacSys_Parts:ASMWL300AFH0E"
 			(at 276.86 147.65 0)
 			(effects
@@
 			)
 		)
-		(property "Footprint" "ASMWLL00NKM0E"
+		(property "Footprint" "SamacSys_Parts:ASMWL300AFH0E"
 			(at 255.27 147.65 0)
 			(effects
@@
 			)
 		)
-		(property "Footprint" "ASMWLL00NKM0E"
+		(property "Footprint" "SamacSys_Parts:ASMWL300AFH0E"
 			(at 213.36 147.65 0)
 			(effects
@@
 			)
 		)
-		(property "Footprint" "ASMWLL00NKM0E"
+		(property "Footprint" "SamacSys_Parts:ASMWLL00NKM0E"
 			(at 257.81 171.78 0)
 			(effects
@@
 			)
 		)
-		(property "Footprint" "ASMWLL00NKM0E"
+		(property "Footprint" "SamacSys_Parts:ASMWLL00NKM0E"
 			(at 279.4 171.78 0)
 			(effects
@@
 			)
 		)
-		(property "Footprint" "SOD3716X145N"
+		(property "Footprint" "SamacSys_Parts:SOD3716X145N"
 			(at 176.53 36.83 0)
 			(effects
@@
 			)
 		)
-		(property "Footprint" "ASMWLL00NKM0E"
+		(property "Footprint" "SamacSys_Parts:ASMWLL00NKM0E"
 			(at 194.31 171.78 0)
 			(effects
@@
 			)
 		)
-		(property "Footprint" "DIOM7959X262N"
+		(property "Footprint" "SamacSys_Parts:DIOM7959X262N"
 			(at 74.93 81.28 0)
 			(effects
@@
 			)
 		)
-		(property "Footprint" "ASMWLL00NKM0E"
+		(property "Footprint" "SamacSys_Parts:ASMWLL00NKM0E"
 			(at 236.22 171.78 0)
 			(effects

Commit message: finished 74 out of 101 footprints
Parts:
- C11, C14, C15, C16, C28, C31, C32, C34, C38, C5, C8: footprint SamacSys_Parts:CAPAE630X800N -> SamacSys_Parts:CAPC1608X90N
- C12, C36: footprint (none) -> SamacSys_Parts:CAPPRD350W60D825H1300
- C13: footprint (none) -> SamacSys_Parts:CAPPRD500W60D1025H1400
- C17, C25, C3, C4: footprint (none) -> SamacSys_Parts:CAPC3216X180N
- C19: footprint (none) -> SamacSys_Parts:0805_AVX
- C20, C21: footprint (none) -> SamacSys_Parts:GRM15x
- C22: footprint (none) -> SamacSys_Parts:CAPC1608X90N
- C24: footprint (none) -> SamacSys_Parts:C0603
- C26: footprint (none) -> SamacSys_Parts:CAPC1005X70N
- C27, C6, C7: footprint (none) -> SamacSys_Parts:CAPC3216X190N
- C29, C37: footprint (none) -> SamacSys_Parts:CAPPRD250W50D655H1250
- C33: footprint (none) -> SamacSys_Parts:CAPC2012X135N
- C9: footprint (none) -> SamacSys_Parts:CAPAE630X800N
- D2: footprint Diode_SMD:D_SMF -> SamacSys_Parts:TVS_SMF12A
- D5, D6, D7: footprint (none) -> LED_THT:LED_D5.0mm
- J1: footprint (none) -> SamacSys_Parts:2828372
- J10: footprint (none) -> Connector_PinHeader_2.54mm:PinHeader_1x12_P2.54mm_Vertical
- J2, J4, J5, J6: footprint (none) -> SamacSys_Parts:691137710003
- J7, J8: footprint (none) -> Connector_PinHeader_2.54mm:PinHeader_1x04_P2.54mm_Vertical
- L1: footprint (none) -> SamacSys_Parts:SRN6045_1
- L2: footprint (none) -> SamacSys_Parts:INDC4949X330N
Changed lines of the file:
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@@
 			)
 		)
-		(property "Footprint" ""
+		(property "Footprint" "SamacSys_Parts:CAPC3216X180N"
 			(at 138.7348 260.35 0)
 			(effects
@@
 			)
 		)
-		(property "Footprint" "SamacSys_Parts:CAPAE630X800N"
+		(property "Footprint" "SamacSys_Parts:CAPC1608X90N"
 			(at 298.1452 199.39 0)
 			(effects
@@
 			)
 		)
-		(property "Footprint" ""
+		(property "Footprint" "SamacSys_Parts:691137710003"
 			(at 77.47 154.94 0)
 			(effects
@@
 			)
 		)
-		(property "Footprint" "SamacSys_Parts:CAPAE630X800N"
+		(property "Footprint" "SamacSys_Parts:CAPC1608X90N"
 			(at 105.1052 41.91 0)
 			(effects
@@
 			)
 		)
-		(property "Footprint" "SamacSys_Parts:CAPAE630X800N"
+		(property "Footprint" "SamacSys_Parts:CAPC1608X90N"
 			(at 92.4052 171.45 0)
 			(effects
@@
 			)
 		)
-		(property "Footprint" ""
+		(property "Footprint" "LED_THT:LED_D5.0mm"
 			(at 316.23 123.19 0)
 			(effects
@@
 			)
 		)
-		(property "Footprint" ""
+		(property "Footprint" "SamacSys_Parts:CAPAE630X800N"
 			(at 83.5152 88.9 0)
 			(effects
@@
 			)
 		)
-		(property "Footprint" "SamacSys_Parts:CAPAE630X800N"
+		(property "Footprint" "SamacSys_Parts:CAPC1608X90N"
 			(at 140.6652 147.32 0)
 			(effects
@@
 			)
 		)
-		(property "Footprint" ""
+		(property "Footprint" "LED_THT:LED_D5.0mm"
 			(at 316.23 100.33 0)
 			(effects
@@
 			)
 		)
-		(property "Footprint" ""
+		(property "Footprint" "LED_THT:LED_D5.0mm"
 			(at 316.23 110.49 0)
 			(effects
@@
 			)
 		)
-		(property "Footprint" "SamacSys_Parts:CAPAE630X800N"
+		(property "Footprint" "SamacSys_Parts:CAPC1608X90N"
 			(at 93.6752 116.84 0)
 			(effects
@@
 			)
 		)
-		(property "Footprint" ""
+		(property "Footprint" "Connector_PinHeader_2.54mm:PinHeader_1x12_P2.54mm_Vertical"
 			(at 335.28 199.39 0)
 			(effects
@@
 			)
 		)
-		(property "Footprint" ""
+		(property "Footprint" "SamacSys_Parts:0805_AVX"
 			(at 73.66 217.4748 0)
 			(effects
@@
 			)
 		)
-		(property "Footprint" ""
+		(property "Footprint" "SamacSys_Parts:GRM15x"
 			(at 145.0848 210.82 0)
 			(effects
@@
 			)
 		)
-		(property "Footprint" ""
+		(property "Footprint" "SamacSys_Parts:CAPC1005X70N"
 			(at 96.52 261.3152 0)
 			(effects
@@
 			)
 		)
-		(property "Footprint" ""
+		(property "Footprint" "SamacSys_Parts:CAPC1608X90N"
 			(at 59.3852 254 0)
 			(effects
@@
 			)
 		)
-		(property "Footprint" ""
+		(property "Footprint" "SamacSys_Parts:2828372"
 			(at 167.64 139.7 0)
 			(effects
@@
 			)
 		)
-		(property "Footprint" "SamacSys_Parts:CAPAE630X800N"
+		(property "Footprint" "SamacSys_Parts:CAPC1608X90N"
 			(at 92.4052 147.32 0)
 			(effects
@@
 			)
 		)
-		(property "Footprint" ""
+		(property "Footprint" "SamacSys_Parts:CAPPRD350W60D825H1300"
 			(at 126.6952 147.32 0)
 			(effects
@@
 			)
 		)
-		(property "Footprint" ""
+		(property "Footprint" "SamacSys_Parts:C0603"
 			(at 122.2248 264.16 0)
 			(effects
@@
 			)
 		)
-		(property "Footprint" ""
+		(property "Footprint" "Connector_PinHeader_2.54mm:PinHeader_1x04_P2.54mm_Vertical"
 			(at 312.42 194.31 0)
 			(effects
@@
 			)
 		)
-		(property "Footprint" ""
+		(property "Footprint" "SamacSys_Parts:691137710003"
 			(at 77.47 172.72 0)
 			(effects
@@
 			)
 		)
-		(property "Footprint" ""
+		(property "Footprint" "SamacSys_Parts:CAPC3216X190N"
 			(at 93.6752 41.91 0)
 			(effects
@@
 			)
 		)
-		(property "Footprint" ""
+		(property "Footprint" "SamacSys_Parts:CAPPRD350W60D825H1300"
 			(at 68.2752 41.91 0)
 			(effects
@@
 			)
 		)
-		(property "Footprint" ""
+		(property "Footprint" "SamacSys_Parts:CAPPRD250W50D655H1250"
 			(at 21.2852 34.29 0)
 			(effects
@@
 			)
 		)
-		(property "Footprint" ""
+		(property "Footprint" "Connector_PinHeader_2.54mm:PinHeader_1x04_P2.54mm_Vertical"
 			(at 339.09 163.83 0)
 			(effects
@@
 			)
 		)
-		(property "Footprint" ""
+		(property "Footprint" "SamacSys_Parts:CAPPRD500W60D1025H1400"
 			(at 138.1252 113.03 0)
 			(effects
@@
 			)
 		)
-		(property "Footprint" ""
+		(property "Footprint" "SamacSys_Parts:CAPPRD250W50D655H1250"
 			(at 31.4452 231.14 0)
 			(effects
@@
 			)
 		)
-		(property "Footprint" ""
+		(property "Footprint" "SamacSys_Parts:SRN6045_1"
 			(at 54.61 218.44 0)
 			(effects
@@
 			)
 		)
-		(property "Footprint" ""
+		(property "Footprint" "SamacSys_Parts:CAPC3216X180N"
 			(at 42.2148 223.52 0)
 			(effects
@@
 			)
 		)
-		(property "Footprint" "SamacSys_Parts:CAPAE630X800N"
+		(property "Footprint" "SamacSys_Parts:CAPC1608X90N"
 			(at 56.8452 34.29 0)
 			(effects
@@
 			)
 		)
-		(property "Footprint" "SamacSys_Parts:CAPAE630X800N"
+		(property "Footprint" "SamacSys_Parts:CAPC1608X90N"
 			(at 125.4252 113.03 0)
 			(effects
@@
 			)
 		)
-		(property "Footprint" ""
+		(property "Footprint" "SamacSys_Parts:691137710003"
 			(at 77.47 113.03 0)
 			(effects
@@
 			)
 		)
-		(property "Footprint" ""
+		(property "Footprint" "SamacSys_Parts:691137710003"
 			(at 173.99 110.49 0)
 			(effects
@@
 			)
 		)
-		(property "Footprint" ""
+		(property "Footprint" "SamacSys_Parts:GRM15x"
 			(at 133.35 193.3448 0)
 			(effects
@@
 			)
 		)
-		(property "Footprint" ""
+		(property "Footprint" "SamacSys_Parts:CAPC3216X180N"
 			(at 33.9852 34.29 0)
 			(effects
@@
 			)
 		)
-		(property "Footprint" ""
+		(property "Footprint" "SamacSys_Parts:CAPC3216X180N"
 			(at 45.4152 34.29 0)
 			(effects
@@
 			)
 		)
-		(property "Footprint" ""
+		(property "Footprint" "SamacSys_Parts:CAPC2012X135N"
 			(at 105.1052 147.32 0)
 			(effects
@@
 			)
 		)
-		(property "Footprint" "SamacSys_Parts:CAPAE630X800N"
+		(property "Footprint" "SamacSys_Parts:CAPC1608X90N"
 			(at 106.3752 88.9 0)
 			(effects
@@
 			)
 		)
-		(property "Footprint" ""
+		(property "Footprint" "SamacSys_Parts:CAPC3216X190N"
 			(at 82.2452 41.91 0)
 			(effects
@@
 			)
 		)
-		(property "Footprint" "SamacSys_Parts:CAPAE630X800N"
+		(property "Footprint" "SamacSys_Parts:CAPC1608X90N"
 			(at 82.2452 133.35 0)
 			(effects
@@
 			)
 		)
-		(property "Footprint" "Diode_SMD:D_SMF"
+		(property "Footprint" "SamacSys_Parts:TVS_SMF12A"
 			(at 62.23 85.09 0)
 			(effects
@@
 			)
 		)
-		(property "Footprint" ""
+		(property "Footprint" "SamacSys_Parts:INDC4949X330N"
 			(at 121.92 31.75 0)
 			(effects
@@
 			)
 		)
-		(property "Footprint" "SamacSys_Parts:CAPAE630X800N"
+		(property "Footprint" "SamacSys_Parts:CAPC1608X90N"
 			(at 302.26 170.4848 0)
 			(effects
@@
 			)
 		)
-		(property "Footprint" ""
+		(property "Footprint" "SamacSys_Parts:CAPC3216X190N"
 			(at 286.7152 199.39 0)
 			(effects

Commit message: most resistor footprints added, need to check
Parts:
- R1, R10, R11, R12, R13, R15, R16, R17, R18, R2, R21, R23, R24, R25, R26, R27, R28, R8, R9: footprint (none) -> SamacSys_Parts:RESC1608X55N
- R19, R20, R4, R5, R6, R7: footprint (none) -> SamacSys_Parts:RESC2012X60N
- R22: footprint (none) -> SamacSys_Parts:RESC3116X65N
- R3: footprint (none) -> Resistor_SMD:R_0805_2012Metric
Changed lines of the file:
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@@
 			)
 		)
-		(property "Footprint" ""
+		(property "Footprint" "SamacSys_Parts:RESC1608X55N"
 			(at 332.74 124.968 90)
 			(effects
@@
 			)
 		)
-		(property "Footprint" ""
+		(property "Footprint" "SamacSys_Parts:RESC1608X55N"
 			(at 161.29 114.808 90)
 			(effects
@@
 			)
 		)
-		(property "Footprint" ""
+		(property "Footprint" "SamacSys_Parts:RESC2012X60N"
 			(at 163.068 36.83 90)
 			(effects
@@
 			)
 		)
-		(property "Footprint" ""
+		(property "Footprint" "SamacSys_Parts:RESC1608X55N"
 			(at 59.182 120.65 90)
 			(effects
@@
 			)
 		)
-		(property "Footprint" ""
+		(property "Footprint" "SamacSys_Parts:RESC1608X55N"
 			(at 331.47 98.552 90)
 			(effects
@@
 			)
 		)
-		(property "Footprint" ""
+		(property "Footprint" "SamacSys_Parts:RESC2012X60N"
 			(at 68.072 237.49 90)
 			(effects
@@
 			)
 		)
-		(property "Footprint" ""
+		(property "Footprint" "SamacSys_Parts:RESC1608X55N"
 			(at 312.42 161.798 90)
 			(effects
@@
 			)
 		)
-		(property "Footprint" ""
+		(property "Footprint" "SamacSys_Parts:RESC1608X55N"
 			(at 331.47 112.268 90)
 			(effects
@@
 			)
 		)
-		(property "Footprint" ""
+		(property "Footprint" "Resistor_SMD:R_0805_2012Metric"
 			(at 163.068 26.67 90)
 			(effects
@@
 			)
 		)
-		(property "Footprint" ""
+		(property "Footprint" "SamacSys_Parts:RESC1608X55N"
 			(at 114.3 274.828 90)
 			(effects
@@
 			)
 		)
-		(property "Footprint" ""
+		(property "Footprint" "SamacSys_Parts:RESC2012X60N"
 			(at 68.072 247.65 90)
 			(effects
@@
 			)
 		)
-		(property "Footprint" ""
+		(property "Footprint" "SamacSys_Parts:RESC3116X65N"
 			(at 68.072 228.6 90)
 			(effects
@@
 			)
 		)
-		(property "Footprint" ""
+		(property "Footprint" "SamacSys_Parts:RESC1608X55N"
 			(at 139.192 237.49 90)
 			(effects
@@
 			)
 		)
-		(property "Footprint" ""
+		(property "Footprint" "SamacSys_Parts:RESC1608X55N"
 			(at 151.892 234.95 90)
 			(effects
@@
 			)
 		)
-		(property "Footprint" ""
+		(property "Footprint" "SamacSys_Parts:RESC1608X55N"
 			(at 144.018 161.29 90)
 			(effects
@@
 			)
 		)
-		(property "Footprint" ""
+		(property "Footprint" "SamacSys_Parts:RESC1608X55N"
 			(at 50.292 171.45 90)
 			(effects
@@
 			)
 		)
-		(property "Footprint" ""
+		(property "Footprint" "SamacSys_Parts:RESC1608X55N"
 			(at 107.95 262.128 90)
 			(effects
@@
 			)
 		)
-		(property "Footprint" ""
+		(property "Footprint" "SamacSys_Parts:RESC1608X55N"
 			(at 59.182 130.81 90)
 			(effects
@@
 			)
 		)
-		(property "Footprint" ""
+		(property "Footprint" "SamacSys_Parts:RESC2012X60N"
 			(at 170.688 36.83 90)
 			(effects
@@
 			)
 		)
-		(property "Footprint" ""
+		(property "Footprint" "SamacSys_Parts:RESC1608X55N"
 			(at 64.008 152.4 90)
 			(effects
@@
 			)
 		)
-		(property "Footprint" ""
+		(property "Footprint" "SamacSys_Parts:RESC2012X60N"
 			(at 113.792 36.83 90)
 			(effects
@@
 			)
 		)
-		(property "Footprint" ""
+		(property "Footprint" "SamacSys_Parts:RESC2012X60N"
 			(at 113.792 46.99 90)
 			(effects
@@
 			)
 		)
-		(property "Footprint" ""
+		(property "Footprint" "SamacSys_Parts:RESC1608X55N"
 			(at 72.39 127.508 90)
 			(effects
@@
 			)
 		)
-		(property "Footprint" ""
+		(property "Footprint" "SamacSys_Parts:RESC1608X55N"
 			(at 149.86 157.988 90)
 			(effects
@@
 			)
 		)
-		(property "Footprint" ""
+		(property "Footprint" "SamacSys_Parts:RESC1608X55N"
 			(at 323.088 153.67 90)
 			(effects
@@
 			)
 		)
-		(property "Footprint" ""
+		(property "Footprint" "SamacSys_Parts:RESC1608X55N"
 			(at 102.87 274.828 90)
 			(effects
@@
 			)
 		)
-		(property "Footprint" ""
+		(property "Footprint" "SamacSys_Parts:RESC1608X55N"
 			(at 133.35 262.128 90)
 			(effects

Commit message: Added level shifter to servo motor, and initiated layout, no routing yet
Parts:
- removed J10: Conn_01x12_Pin, Connector_PinHeader_2.54mm:PinHeader_1x12_P2.54mm_Vertical, symbol Connector:Conn_01x12_Pin
- added C40, C42: 0.1uF, Capacitor_SMD:C_0603_1608Metric, symbol Device:C
- added C43: 4.7uF, Capacitor_SMD:C_1206_3216Metric, symbol Device:C
- added IC5: TXU0101DBVR, SOT95P280X145-6N, symbol SamacSys_Parts:TXU0101DBVR
- added J11: LED Connector, SamacSys_Parts:2828372, symbol Connector:Conn_01x02_Socket
- added J9: Conn_01x10_Pin, Connector_PinHeader_2.54mm:PinHeader_1x10_P2.54mm_Vertical, symbol Connector:Conn_01x10_Pin
- IC1: footprint ESP32WROOM32EN8R2 -> SamacSys_Parts:ESP32WROOM32EN8R2
- IC2: footprint SOT230P700X180-4N -> SamacSys_Parts:SOT230P700X180-4N
- IC3: footprint SOTFL50P160X60-6N -> SamacSys_Parts:SOTFL50P160X60-6N
- IC4: footprint QFN50P400X500X80-29N-D -> SamacSys_Parts:QFN50P400X500X80-29N-D
- Q2: value PMOS -> SI2319CDS-T1-GE3; footprint (none) -> SamacSys_Parts:SOT95P237X112-3N
- R14: footprint (none) -> SamacSys_Parts:CSR1206
- SW1, SW2: footprint (none) -> Button_Switch_SMD:SW_SPST_SKQG_WithStem
Connections:
- net IO17 is gone; now on net PH_FAULT: IC1.28 (IO17)
- net IO32 is gone; now on net FLOW_FAULT: IC1.8 (IO32)
- net IO35 is gone; now on net TEMP_FAULT: IC1.7 (IO35)
- net +3.3V: now also C42.1, IC5.1 (VCCA)
- net +5V: now also C40.1, IC5.5 (OE), IC5.6 (VCCB)
- net FLOW_FAULT: no longer IC1.26 (IO4)
- net GND: now also C40.2, C42.2, C43.2, IC5.2 (GND), J11.2 (Pin_2)
- net IO0: now also IC1.25 (IO0), J9.1 (Pin_1)
- net IO16: now also IC1.27 (IO16), J9.3 (Pin_3)
- net IO19: now also J9.6 (Pin_6)
- net IO2: now also J9.4 (Pin_4)
- net IO21: now also J9.7 (Pin_7)
- net IO22: now also J9.8 (Pin_8)
- net IO4: now also IC1.26 (IO4), J9.2 (Pin_2)
- net IO5: now also J9.5 (Pin_5)
- net ISP: now also C43.1
- net LEDS: now also J11.1 (Pin_1)
- net PH_FAULT: no longer IC1.25 (IO0)
- net SENSOR_VIN: now also J9.10 (Pin_10)
- net SENSOR_VP: now also J9.9 (Pin_9)
- net SRV_SGN: now also IC5.4 (BY)
- net TEMP_FAULT: no longer IC1.27 (IO16)
- new net SRV_SGN_3.3V: IC5.3 (A)

Commit message: added usb-uart programmer so that its easier to program :D
Parts:
- added C44, C46: 4.7uF, Capacitor_SMD:C_0805_2012Metric, symbol Device:C
- added C45, C47: 0.1uF, Capacitor_SMD:C_0603_1608Metric, symbol Device:C
- added D10, D9: LED, LED_SMD:LED_0603_1608Metric, symbol Device:LED
- added D8: SP0503BAHTG, SamacSys_Parts:SP0503BAHTG, symbol SamacSys_Parts:SP0503BAHTG
- added IC6: CP2102C-A01-GQFN28, SamacSys_Parts:QFN50P500X500X80-29N-D, symbol SamacSys_Parts:CP2102C-A01-GQFN28
- added P1: USB_C_Plug_USB2.0, Connector_USB:USB_C_Receptacle_GCT_USB4125-xx-x_6P_TopMnt_Horizontal, symbol Connector:USB_C_Plug_USB2.0
- added Q3, Q4: SS8050, Package_TO_SOT_SMD:SOT-23, symbol Transistor_BJT:SS8050
- added R29, R31: 22.1k, Resistor_SMD:R_0603_1608Metric, symbol Device:R
- added R30: 47.5k, Resistor_SMD:R_0603_1608Metric, symbol Device:R
- added R32, R36, R37: 10k, Resistor_SMD:R_0603_1608Metric, symbol Device:R
- added R33: 5.1k, Resistor_SMD:R_0603_1608Metric, symbol Device:R
- added R34, R35: 1k, SamacSys_Parts:RESC1608X55N, symbol Device:R
- IC5: footprint SOT95P280X145-6N -> SamacSys_Parts:SOT95P280X145-6N
Connections:
- net +3.3V: now also C44.1, C45.1, IC6.6 (VDD), IC6.7 (VREGIN)
- net GND: now also C44.2, C45.2, C46.2, C47.2, D10.1 (K), D8.1 (COMMON_A), D9.1 (K), IC6.29 (GND_2), IC6.3 (GND_1), P1.A1 (GND), P1.A12 (GND), P1.B1 (GND), P1.B12 (GND), P1.S1 (SHIELD), R30.2, R32.2, R33.2
- net IO0: now also Q4.3 (C)
- net MCU_EN: now also Q3.3 (C)
- net RX: now also IC6.25 (RXD), R35.1
- net TX: now also IC6.26 (TXD), R34.1
- new net: P1.A4 (VBUS), P1.A9 (VBUS), P1.B4 (VBUS), P1.B9 (VBUS), R29.1
- new net: IC6.11 (SUSPENDB), R32.1
- new net: IC6.9 (RSTB), R31.1
- new net: Q4.1 (B), R37.2
- new net: D9.2 (A), R34.2
- new net: P1.A5 (CC), R33.1
- new net: D10.2 (A), R35.2
- new net: Q3.1 (B), R36.2
- new net D+: D8.3 (K_2), IC6.4 (D+), P1.A6 (D+)
- new net D-: D8.2 (K_1), IC6.5 (D-), P1.A7 (D-)
- new net DTR: IC6.28 (DTR), Q4.2 (E), R36.1
- new net RTS: IC6.24 (RTS), Q3.2 (E), R37.1
- new net VBUS: C46.1, C47.1, D8.4 (K_3), IC6.8 (VBUS), R29.2, R30.1
- new net VDD: R31.2
- no-connect marks 9 -> 25
Other:
- note added: "DTR = 0, RTS = 1 -> IO0 is pulled down DTR = 1, RTS = 0 -> MCU_EN is pulled down DTR = 0, RTS = 0 -> MCU_EN is pulled high (elsewhere), IO0 is pulled high (internally) DTR = 1, RTS = 1 -> IO0 is pulled high, MCU_EN is pulled high"
- moved on the sheet: C10, C11, C12, C15, C16, C17, C18, C19, C20, C21, C22, C23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

Commit message: modified layout rip
Parts:
- removed C46: 4.7uF, Capacitor_SMD:C_0805_2012Metric, symbol Device:C
- removed C47: 0.1uF, Capacitor_SMD:C_0603_1608Metric, symbol Device:C
- removed D8: SP0503BAHTG, SamacSys_Parts:SP0503BAHTG, symbol SamacSys_Parts:SP0503BAHTG
- removed J9: Conn_01x10_Pin, Connector_PinHeader_2.54mm:PinHeader_1x10_P2.54mm_Vertical, symbol Connector:Conn_01x10_Pin
- added D11, D8: TPD1E05U06QDPYRQ1, SamacSys_Parts:DPY_R-PX1SON-N2_, symbol Diode:1N4148WT
- added D12: TPD1E05U06QDPYRQ1, DPY(R-PX1SON-N2), symbol SamacSys_Parts:TPD1E05U06QDPYRQ1
- added R38, R39: 0, Resistor_SMD:R_0603_1608Metric, symbol Device:R
- C24: footprint SamacSys_Parts:C0603 -> Capacitor_SMD:C_0603_1608Metric
- P1: footprint Connector_USB:USB_C_Receptacle_GCT_USB4125-xx-x_6P_TopMnt_Horizontal -> Connector_USB:USB_C_Receptacle_HRO_TYPE-C-31-M-12
Connections:
- net IO22 is gone; now on net SRV_SGN_3.3V: IC1.36 (IO22)
- net VDD is gone; now on net +3.3V: R31.2
- net +5V: now also P1.A4 (VBUS), P1.A9 (VBUS), P1.B4 (VBUS), P1.B9 (VBUS), R29.1
- net D+: now also D8.1 (K)
- net D-: now also D11.1 (K)
- net FLOW_FAULT: now also IC1.6 (IO34); no longer IC1.8 (IO32)
- net FLOW_SGN: now also IC1.10 (IO25); no longer IC1.11 (IO26)
- net GND: now also D11.2 (A), D8.2 (A); no longer SW1.1
- net PH_SGN: now also IC1.8 (IO32); no longer IC1.6 (IO34)
- net PUMP_SGN: now also IC1.11 (IO26); no longer IC1.10 (IO25)
- net RX: now also R39.2; no longer IC1.34 (RXD0), J7.3 (Pin_3)
- net SRV_SGN: no longer IC1.30 (IO18)
- net TX: now also R38.2; no longer IC1.35 (TXD0), J7.2 (Pin_2)
- net IO16: no longer names the net of IC1.27 (IO16)
- net IO19: no longer names the net of IC1.31 (IO19)
- net IO2: no longer names the net of IC1.24 (IO2)
- net IO21: no longer names the net of IC1.33 (IO21)
- net IO4: no longer names the net of IC1.26 (IO4)
- net IO5: no longer names the net of IC1.29 (IO5)
- new net RXD0: IC1.34 (RXD0), J7.3 (Pin_3), R38.1
- new net TXD0: IC1.35 (TXD0), J7.2 (Pin_2), R39.1
- no-connect marks 25 -> 34
