File: boards/circle_of_life/circle_of_life.kicad_sch (KiCad schematic)
At the start: 131 parts, among them IC1 ESP32-WROOM-32E-N8R2, IC2 TC1262-3.3VDB, IC3 TPS565242DRLR, IC4 LT3922EUFD#PBF, IC5 TXU0101DBVR, IC6 CP2102C-A01-GQFN28, J1 Water Pump Connector, J11 LED Connector, J2 Servo Motor Connector, J3 Power Connector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

Commit message: fixed some footprints
Parts:
- C1, C10, C18, C2, C23, C30, C33, C35, C39, C41: footprint SamacSys_Parts:CAPC2012X135N -> Capacitor_SMD:C_0805_2012Metric
- C11, C14, C15, C16, C28, C31, C32, C34, C38, C5, C8: footprint SamacSys_Parts:CAPC1608X90N -> Capacitor_SMD:C_0805_2012Metric
- C25, C3, C4: footprint SamacSys_Parts:CAPC3216X180N -> Capacitor_SMD:C_0805_2012Metric
- C26: footprint SamacSys_Parts:CAPC1005X70N -> Capacitor_SMD:C_0805_2012Metric
- C40: footprint Capacitor_SMD:C_0603_1608Metric -> Capacitor_SMD:C_0805_2012Metric
Changed lines of the file:
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@@
 			)
 		)
-		(property "Footprint" "SamacSys_Parts:CAPC3216X180N"
+		(property "Footprint" "Capacitor_SMD:C_0805_2012Metric"
 			(at 129.8448 261.62 0)
 			(effects
@@
 			)
 		)
-		(property "Footprint" "SamacSys_Parts:CAPC1608X90N"
+		(property "Footprint" "Capacitor_SMD:C_0805_2012Metric"
 			(at 387.0452 129.54 0)
 			(effects
@@
 			)
 		)
-		(property "Footprint" "SamacSys_Parts:CAPC1608X90N"
+		(property "Footprint" "Capacitor_SMD:C_0805_2012Metric"
 			(at 105.1052 41.91 0)
 			(effects
@@
 			)
 		)
-		(property "Footprint" "SamacSys_Parts:CAPC1608X90N"
+		(property "Footprint" "Capacitor_SMD:C_0805_2012Metric"
 			(at 93.6752 171.45 0)
 			(effects
@@
 			)
 		)
-		(property "Footprint" "SamacSys_Parts:CAPC1608X90N"
+		(property "Footprint" "Capacitor_SMD:C_0805_2012Metric"
 			(at 141.9352 154.94 0)
 			(effects
@@
 			)
 		)
-		(property "Footprint" "SamacSys_Parts:CAPC2012X135N"
+		(property "Footprint" "Capacitor_SMD:C_0805_2012Metric"
 			(at 86.0552 88.9 0)
 			(effects
@@
 			)
 		)
-		(property "Footprint" "SamacSys_Parts:CAPC1608X90N"
+		(property "Footprint" "Capacitor_SMD:C_0805_2012Metric"
 			(at 93.6752 121.92 0)
 			(effects
@@
 			)
 		)
-		(property "Footprint" "SamacSys_Parts:CAPC1005X70N"
+		(property "Footprint" "Capacitor_SMD:C_0805_2012Metric"
 			(at 87.63 262.5852 0)
 			(effects
@@
 			)
 		)
-		(property "Footprint" "SamacSys_Parts:CAPC1608X90N"
+		(property "Footprint" "Capacitor_SMD:C_0805_2012Metric"
 			(at 93.6752 147.32 0)
 			(effects
@@
 			)
 		)
-		(property "Footprint" "SamacSys_Parts:CAPC2012X135N"
+		(property "Footprint" "Capacitor_SMD:C_0805_2012Metric"
 			(at 172.4152 83.82 0)
 			(effects
@@
 			)
 		)
-		(property "Footprint" "SamacSys_Parts:CAPC2012X135N"
+		(property "Footprint" "Capacitor_SMD:C_0805_2012Metric"
 			(at 400.3548 91.44 0)
 			(effects
@@
 			)
 		)
-		(property "Footprint" "Capacitor_SMD:C_0603_1608Metric"
+		(property "Footprint" "Capacitor_SMD:C_0805_2012Metric"
 			(at 263.8552 111.76 0)
 			(effects
@@
 			)
 		)
-		(property "Footprint" "SamacSys_Parts:CAPC1608X90N"
+		(property "Footprint" "Capacitor_SMD:C_0805_2012Metric"
 			(at 56.8452 34.29 0)
 			(effects
@@
 			)
 		)
-		(property "Footprint" "SamacSys_Parts:CAPC1608X90N"
+		(property "Footprint" "Capacitor_SMD:C_0805_2012Metric"
 			(at 125.4252 113.03 0)
 			(effects
@@
 			)
 		)
-		(property "Footprint" "SamacSys_Parts:CAPC2012X135N"
+		(property "Footprint" "Capacitor_SMD:C_0805_2012Metric"
 			(at 106.3752 121.92 0)
 			(effects
@@
 			)
 		)
-		(property "Footprint" "SamacSys_Parts:CAPC2012X135N"
+		(property "Footprint" "Capacitor_SMD:C_0805_2012Metric"
 			(at 183.8452 83.82 0)
 			(effects
@@
 			)
 		)
-		(property "Footprint" "SamacSys_Parts:CAPC2012X135N"
+		(property "Footprint" "Capacitor_SMD:C_0805_2012Metric"
 			(at 44.7548 224.79 0)
 			(effects
@@
 			)
 		)
-		(property "Footprint" "SamacSys_Parts:CAPC3216X180N"
+		(property "Footprint" "Capacitor_SMD:C_0805_2012Metric"
 			(at 33.9852 34.29 0)
 			(effects
@@
 			)
 		)
-		(property "Footprint" "SamacSys_Parts:CAPC3216X180N"
+		(property "Footprint" "Capacitor_SMD:C_0805_2012Metric"
 			(at 45.4152 34.29 0)
 			(effects
@@
 			)
 		)
-		(property "Footprint" "SamacSys_Parts:CAPC2012X135N"
+		(property "Footprint" "Capacitor_SMD:C_0805_2012Metric"
 			(at 106.3752 147.32 0)
 			(effects
@@
 			)
 		)
-		(property "Footprint" "SamacSys_Parts:CAPC2012X135N"
+		(property "Footprint" "Capacitor_SMD:C_0805_2012Metric"
 			(at 76.5048 234.95 0)
 			(effects
@@
 			)
 		)
-		(property "Footprint" "SamacSys_Parts:CAPC1608X90N"
+		(property "Footprint" "Capacitor_SMD:C_0805_2012Metric"
 			(at 96.2152 88.9 0)
 			(effects
@@
 			)
 		)
-		(property "Footprint" "SamacSys_Parts:CAPC1608X90N"
+		(property "Footprint" "Capacitor_SMD:C_0805_2012Metric"
 			(at 60.6552 133.35 0)
 			(effects
@@
 			)
 		)
-		(property "Footprint" "SamacSys_Parts:CAPC2012X135N"
+		(property "Footprint" "Capacitor_SMD:C_0805_2012Metric"
 			(at 457.5048 90.17 0)
 			(effects
@@
 			)
 		)
-		(property "Footprint" "SamacSys_Parts:CAPC1608X90N"
+		(property "Footprint" "Capacitor_SMD:C_0805_2012Metric"
 			(at 382.27 99.3648 0)
 			(effects
@@
 			)
 		)
-		(property "Footprint" "SamacSys_Parts:CAPC2012X135N"
+		(property "Footprint" "Capacitor_SMD:C_0805_2012Metric"
 			(at 106.3752 171.45 0)
 			(effects

Commit message: fixed most of the footprints errors
Parts:
- D12: footprint DPY(R-PX1SON-N2) -> SamacSys_Parts:DPY_R-PX1SON-N2_
Changed lines of the file:
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@@
 			)
 		)
-		(property "Footprint" "DPY(R-PX1SON-N2)"
+		(property "Footprint" "SamacSys_Parts:DPY_R-PX1SON-N2_"
 			(at 342.9 265.1 0)
 			(effects

Commit message: Fixed DRC for main board
Parts:
- removed D12: TPD1E05U06QDPYRQ1, SamacSys_Parts:DPY_R-PX1SON-N2_, symbol SamacSys_Parts:TPD1E05U06QDPYRQ1
- removed LED1, LED10, LED3, LED5, LED9: ASMW-LL00-NKM0E, SamacSys_Parts:ASMWLL00NKM0E, symbol SamacSys_Parts:ASMW-LL00-NKM0E
- removed LED2, LED4, LED6, LED7, LED8: ASMW-LD00-AGJ0E, SamacSys_Parts:ASMWL300AFH0E, symbol SamacSys_Parts:ASMW-LL00-NKM0E
Other:
- note removed: "Deep Red: 2.25 Vf, 200-300mA Royal Blue: 3.08 VF, 200-300mA"

Commit message: modified some wrong values in led driver
Parts:
- removed C25: 10uF, Capacitor_SMD:C_0805_2012Metric, symbol Device:C
- removed R17: 10k, SamacSys_Parts:RESC1608X55N, symbol Device:R
- R1: value 220 -> 47
- R18: value 499k -> 45.3k
Connections:
- no-connect marks 34 -> 35
Other:
- note removed: "Need to double check and take notes of ALL VALUES"
- moved on the sheet: C1, C10, C11, C12, C13, C14, C15, C16, C17, C18, C19, C2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

Commit message: changed value
Parts:
- R21: value 100M -> 1M
Changed lines of the file:
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@@
 			)
 		)
-		(property "Value" "100M"
+		(property "Value" "1M"
 			(at 287.02 101.6 90)
 			(effects
