File: boards/grow_lights/grow_lights.kicad_sch (KiCad schematic)
At the start: 11 parts, among them J11 LED Connector

Commit message: updated grow lights board with wider traces & removed power plane
Connections:
- net GND is gone; now on net LED-: LED10.2 (K)
Changed lines of the file:
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@@
 		(on_board yes)
 		(dnp no)
-		(fields_autoplaced yes)
 		(property "Reference" "#PWR062"
 			(at 209.55 86.36 0)
@@
 			)
 		)
-		(property "Value" "GND"
+		(property "Value" "LED-"
 			(at 209.55 85.09 0)
 			(effects

Commit message: grow lights PCB
Parts:
- added H1, H2, H3, H4: MountingHole, MountingHole:MountingHole_3.2mm_M3, symbol Mechanical:MountingHole

Commit message: code and grow lights pcb updates
Parts:
- LED2, LED4, LED6, LED7, LED8: footprint SamacSys_Parts:ASMWL300AFH0E -> SamacSys_Parts:ASMWLL00NKM0E
Changed lines of the file:
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@@
 			)
 		)
-		(property "Footprint" "SamacSys_Parts:ASMWL300AFH0E"
+		(property "Footprint" "SamacSys_Parts:ASMWLL00NKM0E"
 			(at 152.4 -37.77 0)
 			(effects
@@
 			)
 		)
-		(property "Footprint" "SamacSys_Parts:ASMWL300AFH0E"
+		(property "Footprint" "SamacSys_Parts:ASMWLL00NKM0E"
 			(at 111.76 -37.77 0)
 			(effects
@@
 			)
 		)
-		(property "Footprint" "SamacSys_Parts:ASMWL300AFH0E"
+		(property "Footprint" "SamacSys_Parts:ASMWLL00NKM0E"
 			(at 194.31 -37.77 0)
 			(effects
@@
 			)
 		)
-		(property "Footprint" "SamacSys_Parts:ASMWL300AFH0E"
+		(property "Footprint" "SamacSys_Parts:ASMWLL00NKM0E"
 			(at 172.72 -37.77 0)
 			(effects
@@
 			)
 		)
-		(property "Footprint" "SamacSys_Parts:ASMWL300AFH0E"
+		(property "Footprint" "SamacSys_Parts:ASMWLL00NKM0E"
 			(at 130.81 -37.77 0)
 			(effects
